File: APPS:ETC/APPS:ETC.kicad_sch (KiCad schematic)
At the start: 6 parts, among them U1 NUCLEO-L432KC, U2 ISO1050DUB, U3 A1365xKTTN-1, U4 A1365xKTTN-1, U5 L78S05CV

Commit message: adding more stuff
schema
Parts:
- added C2: C- 0.1microF, symbol Device:C
Connections:
- net +5V: now also C2.2
Changed lines of the file:
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@@
   (junction (at 76.2 39.37) (diameter 0) (color 0 0 0 0)
+  )
+  (junction (at 139.7 29.21) (diameter 0) (color 0 0 0 0)
   )
   (junction (at 163.83 49.53) (diameter 0) (color 0 0 0 0)
@@
     (stroke (width 0) (type default))
   )
+  (wire (pts (xy 88.9 31.75) (xy 88.9 48.26))
+    (stroke (width 0) (type default))
+  )
   (wire (pts (xy 144.78 74.93) (xy 144.78 92.71))
     (stroke (width 0) (type default))
@@
     (stroke (width 0) (type default))
   )
+  (wire (pts (xy 137.16 48.26) (xy 137.16 29.21))
+    (stroke (width 0) (type default))
+  )
+  (wire (pts (xy 139.7 29.21) (xy 142.24 29.21))
+    (stroke (width 0) (type default))
+  )
   (wire (pts (xy 73.66 24.13) (xy 76.2 24.13))
     (stroke (width 0) (type default))
   )
   (wire (pts (xy 191.77 82.55) (xy 193.04 82.55))
+    (stroke (width 0) (type default))
+  )
+  (wire (pts (xy 128.27 72.39) (xy 139.7 72.39))
     (stroke (width 0) (type default))
   )
@@
     (stroke (width 0) (type default))
   )
-  (wire (pts (xy 137.16 29.21) (xy 142.24 29.21))
-    (stroke (width 0) (type default))
-  )
-  (wire (pts (xy 134.62 29.21) (xy 134.62 72.39))
+  (wire (pts (xy 137.16 29.21) (xy 139.7 29.21))
     (stroke (width 0) (type default))
   )
@@
   )
   (wire (pts (xy 82.55 24.13) (xy 82.55 29.21))
+    (stroke (width 0) (type default))
+  )
+  (wire (pts (xy 113.03 48.26) (xy 137.16 48.26))
     (stroke (width 0) (type default))
   )
@@
     (stroke (width 0) (type default))
   )
-  (wire (pts (xy 134.62 72.39) (xy 128.27 72.39))
+  (wire (pts (xy 88.9 48.26) (xy 105.41 48.26))
     (stroke (width 0) (type default))
   )
+  (wire (pts (xy 139.7 29.21) (xy 139.7 72.39))
+    (stroke (width 0) (type default))
+  )
+  (symbol (lib_id "Device:C") (at 109.22 48.26 90) (unit 1)
+    (in_bom yes) (on_board yes) (dnp no) (fields_autoplaced)
+    (property "Reference" "C2" (at 109.22 40.64 90)
+      (effects (font (size 1.27 1.27)))
+    )
+    (property "Value" "C- 0.1microF" (at 109.22 43.18 90)
+      (effects (font (size 1.27 1.27)))
+    )
+    (property "Footprint" "" (at 113.03 47.2948 0)
+      (effects (font (size 1.27 1.27)) hide)
+    )
+    (property "Datasheet" "~" (at 109.22 48.26 0)
+      (effects (font (size 1.27 1.27)) hide)
+    )
+    (pin "1")
+    (pin "2")
+    (instances
+      (project "APPS:ETC"
+        (path "/21da8b0a-bf7f-4003-9579-5de7190091be"
+          (reference "C2") (unit 1)
+        )
+      )
+    )
+  )
   (symbol (lib_id "power:Earth") (at 130.81 67.31 90) (unit 1)
