File: APPS_ETCA/APPS_ETC.kicad_pcb (KiCad board)
At the start: 2 copper layers, 21 parts, among them P1 DTM1312PC12PDR008, U1 NSL-32, U2 DK1A1B-12V, U3 MCP6004, U6 LM7805_TO220, U8 LM7809_TO220

Commit message: board layout w connectors
Parts:
- moved U3 165.4 mm to (231.1, 66.0)
- moved R5 162.6 mm to (249.9, 51.6)
- moved R7 162.5 mm to (232.7, 45.7)
- moved STM-32_Microcontroller1 154.8 mm to (210.8, 77.2)
- moved R4 115.9 mm to (223.1, 116.8)
- moved R3 115.5 mm to (222.5, 111.8)
- moved U2 112.2 mm to (177.8, 48.3)
- moved R2 105.9 mm to (212.9, 109.2)
- moved U1 89.7 mm to (207.9, 115.5)
- moved U6 76.2 mm to (193.0, 109.2)
- moved U8 58.4 mm to (175.3, 116.8)
- moved D1 58.0 mm to (172.7, 101.6)
- moved CAN_Tranceiver1 48.5 mm to (190.5, 91.4)
- moved C5 44.5 mm to (150.9, 83.8)
- moved C2 40.8 mm to (143.3, 68.6)
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Connections:
- P1 pad C1: Sound -> OUT2
- P1 pad C2: Green -> OUT1
- P1 pad C3: CANL -> GND
- P1 pad C4: CANH -> 5V
- P1 pad C6: 12V -> 5V
- P1 pad D1: OUT2 -> Sound
- P1 pad D2: OUT1 -> Green
- P1 pad D3: GND -> CANL
- P1 pad D4: GND -> CANH
- P1 pad D5: 5V -> GND
- P1 pad D6: 5V -> 12V
Routing:
- net unconnected-(P1-PadC7): track 0.00 -> 11.5 mm

Commit message: updated schema
Parts:
- added CR1: STS6NF20V, 1FS_2_Global_Footprint_Library:SOIC127P600X175-8N, F.Cu at (180.3, 76.2)
- moved U3 9.25 mm to (240.0, 63.5)
Connections:
- net 3V renamed +3.3V
- net CANH renamed /CANH
- net CANL renamed /CANL
- net D10 OUT renamed /D10 OUT
- net D2 OUT renamed /D2 OUT
- C3 pad 2: Earth -> GND
- CAN_Tranceiver1 pad 4: Earth -> GND
- CAN_Tranceiver1 pad 8: 5V -> +5V
- P1 pad C1: OUT2 -> unconnected-(P1-PadC1)
- P1 pad C11: unconnected-(P1-PadC11) -> GND
- P1 pad C12: unconnected-(P1-PadC12) -> +5V
- P1 pad C2: OUT1 -> unconnected-(P1-PadC2)
- P1 pad C3: GND -> unconnected-(P1-PadC3)
- P1 pad C4: 5V -> unconnected-(P1-PadC4)
- P1 pad C5: GND -> unconnected-(P1-PadC5)
- P1 pad C6: 5V -> unconnected-(P1-PadC6)
- P1 pad C7: unconnected-(P1-PadC7) -> /OUT2
- P1 pad C8: unconnected-(P1-PadC8) -> GND
- P1 pad C9: unconnected-(P1-PadC9) -> +5V
- P1 pad D1: Sound -> /RTDS GND
- P1 pad D2: Green -> +12V
- P1 pad D6: 12V -> +12V
- P1 pad D7: unconnected-(P1-PadD7) -> /Brake Sensor
- STM-32_Microcontroller1 pad CN3_10: RTDS -> /RTDS Control
- STM-32_Microcontroller1 pad CN3_6: unconnected-(STM-32_Microcontroller1A-PB0-PadCN3_6) -> /LED
- STM-32_Microcontroller1 pad CN3_9: TSAL -> unconnected-(STM-32_Microcontroller1A-PB1-PadCN3_9)
- STM-32_Microcontroller1 pad CN4_10: unconnected-(STM-32_Microcontroller1A-PA3-PadCN4_10) -> /Brake Sensor
- U3 pad 2: OUT1 -> /OUT1
- U3 pad 6: OUT2 -> /OUT2
Routing:
- net unconnected-(P1-PadC7): track 11.5 -> 0.00 mm

Commit message: for my colead abhi <3
Parts:
- removed D1: D, Diode_THT:D_DO-41_SOD81_P10.16mm_Horizontal
- added R6: 10 ohm, Resistor_SMD:R_0805_2012Metric_Pad1.20x1.40mm_HandSolder, F.Cu at (157.3, 104.4)
- moved C1 122.2 mm to (241.3, 119.9)
- moved C2 115.6 mm to (246.9, 119.9), turned to 180 degrees
- moved C6 110.1 mm to (233.7, 119.9), turned to 180 degrees
- moved C5 86.1 mm to (229.1, 119.9)
- moved R1 79.0 mm to (212.4, 66.0)
- moved U1 58.3 mm to (150.1, 107.9)
- moved U8 53.9 mm to (229.1, 114.8)
- moved U6 47.6 mm to (240.3, 114.8)
- moved CAN_Tranceiver1 34.6 mm to (214.3, 116.6)
- moved R3 33.1 mm to (220.0, 78.7)
- moved U2 31.0 mm to (152.4, 30.5)
- moved CR1 29.6 mm to (154.9, 61.0)
- moved STM-32_Microcontroller1 22.9 mm to (188.0, 76.2)
- moved R2 19.0 mm to (207.8, 90.9)
- moved R4 19.0 mm to (217.9, 98.6)
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Routing:
- net GND: track 0.00 -> 115.0 mm
- net +12V: track 0.00 -> 37.4 mm
- net +9V: track 0.00 -> 5.31 mm
Other:
- board outline added: 81.3 x 99.1 mm

Commit message: Linear Reg. CAN. All that
Parts:
- moved C4 99.1 mm to (220.5, 120.4), turned to -90 degrees
- moved R5 73.7 mm to (223.5, 120.4), turned to -90 degrees
- moved CAN_Tranceiver1 5.55 mm to (208.8, 116.8)
Connections:
- P1 pad C10: unconnected-(P1-PadC10) -> /OUT1
Routing:
- net +5V: track 0.00 -> 84.8 mm
- net /CANH: track 0.00 -> 31.4 mm
- net /CANL: track 0.00 -> 26.2 mm
- net GND: track 115.0 -> 141.0 mm, vias 0 -> 2
- net +12V: track 37.4 -> 56.6 mm

Commit message: thug changes
Parts:
- removed U1: NSL-32, 1FS_2_Global_Footprint_Library:OptoCoupler 6-SOP
- removed U2: DK1A1B-12V, 1FS_2_Global_Footprint_Library:RELAY_DK2A_PAN
- moved C3 82.7 mm to (197.1, 118.4), turned to -90 degrees
Routing:
- net +3.3V: track 0.00 -> 9.82 mm, vias 0 -> 2
- net GND: track 141.0 -> 146.8 mm

Commit message: for my pcb/coding/schema master dwang
Parts:
- moved R2 20.0 mm to (210.8, 71.1)
- moved R4 14.7 mm to (218.4, 83.8)
Routing:
- net Net-(U3A-+): track 0.00 -> 41.8 mm
- net Net-(U3B-+): track 0.00 -> 31.1 mm, vias 0 -> 3
- net Net-(STM-32_Microcontroller1A-PA0): track 0.00 -> 30.1 mm
- net Net-(STM-32_Microcontroller1A-PA1): track 0.00 -> 26.7 mm
Changed lines of the file:
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@@
     (property "ki_keywords" "R res resistor")
     (attr smd)
-    (fp_text reference "R3" (at -2 -6.32) (layer "F.SilkS")
-        (effects (font (size 1 1) (thickness 0.15)))
-    )
-    (fp_text value "180kO" (at 0 1.65) (layer "F.Fab")
-        (effects (font (size 1 1) (thickness 0.15)))
-    )
-    (fp_text user "${REFERENCE}" (at -2 -4.67) (layer "F.Fab")
+    (fp_text reference "R3" (at 1 -2.54) (layer "F.SilkS")
+        (effects (font (size 1 1) (thickness 0.15)))
+    )
+    (fp_text value "180kO" (at 0 1.65) (layer "F.Fab") hide
+        (effects (font (size 1 1) (thickness 0.15)))
+    )
+    (fp_text user "${REFERENCE}" (at 0 -0.625) (layer "F.Fab")
         (effects (font (size 0.5 0.5) (thickness 0.08)))
     )
@@
   )
   (footprint "Resistor_SMD:R_0805_2012Metric_Pad1.20x1.40mm_HandSolder" (layer "F.Cu")
-    (at 207.788 90.932)
+    (at 210.82 71.12)
     (descr "Resistor SMD 0805 (2012 Metric), square (rectangular) end terminal, IPC_7351 nominal with elongated pad for handsoldering. (Body size source: IPC-SM-782 page 72, https://www.pcb-3d.com/wordpress/wp-content/uploads/ipc-sm-782a_amendment_1_and_2.pdf), generated with kicad-footprint-generator")
     (tags "resistor handsolder")
@@
   )
   (footprint "Resistor_SMD:R_0805_2012Metric_Pad1.20x1.40mm_HandSolder" (layer "F.Cu")
-    (at 217.948 98.552)
+    (at 218.44 83.82)
     (descr "Resistor SMD 0805 (2012 Metric), square (rectangular) end terminal, IPC_7351 nominal with elongated pad for handsoldering. (Body size source: IPC-SM-782 page 72, https://www.pcb-3d.com/wordpress/wp-content/uploads/ipc-sm-782a_amendment_1_and_2.pdf), generated with kicad-footprint-generator")
     (tags "resistor handsolder")
@@
   (segment (start 234.739 115.359) (end 234.188 114.808) (width 0.25) (layer "F.Cu") (net 13))
   (segment (start 234.739 119.888) (end 234.739 115.359) (width 0.25) (layer "F.Cu") (net 13))
-  (segment (start 172.97 114.55) (end 172.72 114.3) (width 0.25) (layer "F.Cu") (net 18))
+  (segment (start 218.44 60.96) (end 223.52 66.04) (width 0.25) (layer "F.Cu") (net 14))
+  (segment (start 233.68 60.96) (end 216.44 60.96) (width 0.25) (layer "F.Cu") (net 14))
+  (segment (start 223.52 66.04) (end 233.68 66.04) (width 0.25) (layer "F.Cu") (net 14))
+  (segment (start 216.44 60.96) (end 211.36 66.04) (width 0.25) (layer "F.Cu") (net 14))
+  (segment (start 209.82 71.12) (end 209.82 71.145) (width 0.25) (layer "F.Cu") (net 15))
+  (segment (start 213.36 66.04) (end 213.36 67.58) (width 0.25) (layer "F.Cu") (net 15))
+  (segment (start 209.82 71.145) (end 195.58 85.385) (width 0.25) (layer "F.Cu") (net 15))
+  (segment (start 213.36 67.58) (end 209.82 71.12) (width 0.25) (layer "F.Cu") (net 15))
+  (segment (start 233.68 76.2) (end 231.14 76.2) (width 0.25) (layer "F.Cu") (net 16))
+  (segment (start 233.68 71.12) (end 226.06 71.12) (width 0.25) (layer "F.Cu") (net 16))
+  (segment (start 226.06 71.12) (end 220.98 76.2) (width 0.25) (layer "F.Cu") (net 16))
+  (segment (start 231.14 76.2) (end 228.6 76.2) (width 0.25) (layer "F.Cu") (net 16))
+  (via (at 226.06 71.12) (size 0.8) (drill 0.4) (layers "F.Cu" "B.Cu") (net 16))
+  (via (at 228.6 76.2) (size 0.8) (drill 0.4) (layers "F.Cu" "B.Cu") (net 16))
+  (via (at 231.14 76.2) (size 0.8) (drill 0.4) (layers "F.Cu" "B.Cu") (net 16))
+  (segment (start 220.98 76.2) (end 218.44 78.74) (width 0.25) (layer "B.Cu") (net 16))
+  (segment (start 228.6 76.2) (end 220.98 76.2) (width 0.25) (layer "B.Cu") (net 16))
+  (segment (start 217.44 83.82) (end 199.685 83.82) (width 0.25) (layer "F.Cu") (net 17))
+  (segment (start 199.685 83.82) (end 195.58 87.925) (width 0.25) (layer "F.Cu") (net 17))
+  (segment (start 220.98 78.74) (end 220.98 80.28) (width 0.25) (layer "F.Cu") (net 17))
+  (segment (start 220.98 80.28) (end 217.44 83.82) (width 0.25) (layer "F.Cu") (net 17))
 )
