File: APPS_ETCA/APPS_ETC.kicad_pcb (KiCad board)
At the start: 2 copper layers, 81.3 x 99.1 mm, 20 parts, among them P1 DTM1312PC12PDR008, U3 MCP6004, U6 LM7805_TO220, U8 LM7809_TO220

Commit message: MORE
Parts:
- removed R7: 480, Resistor_SMD:R_0805_2012Metric_Pad1.20x1.40mm_HandSolder
- moved CR1 64.8 mm to (189.5, 115.8), turned to 180 degrees
Routing:
- net /D2 OUT: track 0.00 -> 69.9 mm, vias 0 -> 2
- net /RTDS GND: track 0.00 -> 48.6 mm, vias 0 -> 2
- net /D10 OUT: track 0.00 -> 44.9 mm
- net /RTDS Control: track 0.00 -> 40.8 mm
- net GND: track 146.8 -> 154.9 mm

Commit message: MOREEE
Routing:
- net +5V: track 84.8 -> 120.3 mm
Changed lines of the file:
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@@
   (via (at 194.564 119.38) (size 0.8) (drill 0.4) (layers "F.Cu" "B.Cu") (net 9))
   (segment (start 194.564 119.38) (end 187.96 119.38) (width 0.25) (layer "B.Cu") (net 9))
+  (segment (start 243.84 111.252) (end 245.364 112.776) (width 0.25) (layer "F.Cu") (net 10))
+  (segment (start 224.282 113.03) (end 226.06 111.252) (width 0.25) (layer "F.Cu") (net 10))
   (segment (start 245.364 117.348) (end 247.904 119.888) (width 0.25) (layer "F.Cu") (net 10))
+  (segment (start 213.313 113.03) (end 224.282 113.03) (width 0.25) (layer "F.Cu") (net 10))
+  (segment (start 226.06 111.252) (end 243.84 111.252) (width 0.25) (layer "F.Cu") (net 10))
   (segment (start 245.364 114.808) (end 245.364 117.348) (width 0.25) (layer "F.Cu") (net 10))
+  (segment (start 245.364 112.776) (end 245.364 114.808) (width 0.25) (layer "F.Cu") (net 10))
   (segment (start 245.364 114.808) (end 245.364 113.792) (width 0.25) (layer "B.Cu") (net 10))
   (segment (start 199.195 120.455) (end 193.92 125.73) (width 0.25) (layer "B.Cu") (net 10))

Commit message: pcb making progress :D
Routing:
- net GND: track 154.9 -> 386.9 mm
- net +3.3V: track 9.82 -> 34.0 mm
Changed lines of the file:
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@@
   (via (at 214.884 121.412) (size 0.8) (drill 0.4) (layers "F.Cu" "B.Cu") (net 2))
   (segment (start 214.884 126.747) (end 215.392 127.255) (width 0.25) (layer "B.Cu") (net 2))
+  (segment (start 241.3 68.58) (end 245.745 68.58) (width 0.25) (layer "B.Cu") (net 2))
   (segment (start 214.884 122.936) (end 214.376 123.444) (width 0.25) (layer "B.Cu") (net 2))
+  (segment (start 180.34 67.605) (end 173.015 67.605) (width 0.25) (layer "B.Cu") (net 2))
+  (segment (start 173.355 57.15) (end 170.815 54.61) (width 0.25) (layer "B.Cu") (net 2))
+  (segment (start 248.54 129.54) (end 249.175 128.905) (width 0.25) (layer "B.Cu") (net 2))
+  (segment (start 175.895 125.73) (end 172.72 128.905) (width 0.25) (layer "B.Cu") (net 2))
+  (segment (start 170.815 57.15) (end 170.815 53.975) (width 0.25) (layer "B.Cu") (net 2))
+  (segment (start 244.73 125.73) (end 248.54 129.54) (width 0.25) (layer "B.Cu") (net 2))
+  (segment (start 172.72 128.905) (end 172.085 128.905) (width 0.25) (layer "B.Cu") (net 2))
   (segment (start 243.205 127.255) (end 244.73 125.73) (width 0.25) (layer "B.Cu") (net 2))
+  (segment (start 249.175 128.905) (end 250.19 128.905) (width 0.25) (layer "B.Cu") (net 2))
+  (segment (start 184.785 57.15) (end 173.355 57.15) (width 0.25) (layer "B.Cu") (net 2))
+  (segment (start 171.11 67.605) (end 170.815 67.31) (width 0.25) (layer "B.Cu") (net 2))
   (segment (start 242.824 113.792) (end 242.824 114.808) (width 0.25) (layer "B.Cu") (net 2))
   (segment (start 232.664 112.776) (end 241.808 112.776) (width 0.25) (layer "B.Cu") (net 2))
+  (segment (start 172.085 128.905) (end 170.815 127.635) (width 0.25) (layer "B.Cu") (net 2))
+  (segment (start 170.815 78.105) (end 170.815 67.31) (width 0.25) (layer "B.Cu") (net 2))
   (segment (start 214.884 123.952) (end 214.884 126.747) (width 0.25) (layer "B.Cu") (net 2))
+  (segment (start 248.285 66.04) (end 248.285 45.72) (width 0.25) (layer "B.Cu") (net 2))
   (segment (start 178.679881 127.249881) (end 177.16 125.73) (width 0.25) (layer "B.Cu") (net 2))
   (segment (start 214.376 123.444) (end 201.676 123.444) (width 0.25) (layer "B.Cu") (net 2))
+  (segment (start 170.815 53.975) (end 170.815 44.45) (width 0.25) (layer "B.Cu") (net 2))
+  (segment (start 170.815 54.61) (end 170.815 53.975) (width 0.25) (layer "B.Cu") (net 2))
   (segment (start 214.376 123.444) (end 214.884 123.952) (width 0.25) (layer "B.Cu") (net 2))
   (segment (start 214.884 122.936) (end 214.884 123.952) (width 0.25) (layer "B.Cu") (net 2))
+  (segment (start 177.16 125.73) (end 175.895 125.73) (width 0.25) (layer "B.Cu") (net 2))
+  (segment (start 170.815 65.405) (end 170.815 57.15) (width 0.25) (layer "B.Cu") (net 2))
   (segment (start 214.884 121.412) (end 214.884 122.936) (width 0.25) (layer "B.Cu") (net 2))
   (segment (start 191.255 127.255) (end 214.376 127.255) (width 0.25) (layer "B.Cu") (net 2))
@@
   (segment (start 241.808 112.776) (end 242.824 113.792) (width 0.25) (layer "B.Cu") (net 2))
   (segment (start 201.168 122.936) (end 201.168 121.412) (width 0.25) (layer "B.Cu") (net 2))
+  (segment (start 170.815 127.635) (end 170.815 78.105) (width 0.25) (layer "B.Cu") (net 2))
   (segment (start 214.376 127.255) (end 215.392 127.255) (width 0.25) (layer "B.Cu") (net 2))
   (segment (start 214.884 126.747) (end 214.376 127.255) (width 0.25) (layer "B.Cu") (net 2))
+  (segment (start 250.19 128.905) (end 250.825 129.54) (width 0.25) (layer "B.Cu") (net 2))
   (segment (start 189.73 125.73) (end 191.255 127.255) (width 0.25) (layer "B.Cu") (net 2))
+  (segment (start 250.825 100.33) (end 248.285 97.79) (width 0.25) (layer "B.Cu") (net 2))
+  (segment (start 170.815 67.31) (end 170.815 65.405) (width 0.25) (layer "B.Cu") (net 2))
   (segment (start 189.73 125.73) (end 188.210119 127.249881) (width 0.25) (layer "B.Cu") (net 2))
   (segment (start 188.210119 127.249881) (end 178.679881 127.249881) (width 0.25) (layer "B.Cu") (net 2))
+  (segment (start 248.285 97.79) (end 248.285 66.04) (width 0.25) (layer "B.Cu") (net 2))
+  (segment (start 195.58 62.525) (end 190.16 62.525) (width 0.25) (layer "B.Cu") (net 2))
   (segment (start 231.648 113.792) (end 232.664 112.776) (width 0.25) (layer "B.Cu") (net 2))
+  (segment (start 190.16 62.525) (end 184.785 57.15) (width 0.25) (layer "B.Cu") (net 2))
+  (segment (start 245.745 68.58) (end 248.285 66.04) (width 0.25) (layer "B.Cu") (net 2))
+  (segment (start 250.825 129.54) (end 250.825 100.33) (width 0.25) (layer "B.Cu") (net 2))
   (segment (start 215.392 127.255) (end 243.205 127.255) (width 0.25) (layer "B.Cu") (net 2))
+  (segment (start 173.015 67.605) (end 170.815 65.405) (width 0.25) (layer "B.Cu") (net 2))
+  (segment (start 196.51 93.005) (end 198.755 95.25) (width 0.25) (layer "F.Cu") (net 3))
   (segment (start 197.104 117.3265) (end 197.104 115.824) (width 0.25) (layer "F.Cu") (net 3))
   (segment (start 204.009 113.284) (end 204.263 113.03) (width 0.25) (layer "F.Cu") (net 3))
+  (segment (start 198.755 95.25) (end 198.755 107.522) (width 0.25) (layer "F.Cu") (net 3))
+  (segment (start 198.755 107.522) (end 204.263 113.03) (width 0.25) (layer "F.Cu") (net 3))
   (segment (start 202.184 113.284) (end 204.009 113.284) (width 0.25) (layer "F.Cu") (net 3))
+  (segment (start 195.58 93.005) (end 196.51 93.005) (width 0.25) (layer "F.Cu") (net 3))
   (via (at 197.104 115.824) (size 0.8) (drill 0.4) (layers "F.Cu" "B.Cu") (net 3))
   (via (at 202.184 113.284) (size 0.8) (drill 0.4) (layers "F.Cu" "B.Cu") (net 3))

Commit message: LEGGO
Parts:
- removed STM-32_Microcontroller1: NUCLEO-L432KC, 1FS_2_Global_Footprint_Library:MODULE_NUCLEO-L432KC
- removed U3: MCP6004, FSFootprints:PDIP14_300MC_MCH
- added R7: 180kO, Resistor_SMD:R_0805_2012Metric_Pad1.20x1.40mm_HandSolder, F.Cu at (221.5, 85.4)
- added R8: 330kO, Resistor_SMD:R_0805_2012Metric_Pad1.20x1.40mm_HandSolder, F.Cu at (221.5, 90.4)
- added U1: NUCLEO-L432KC, 1FS_2_Global_Footprint_Library:MODULE_NUCLEO-L432KC, F.Cu at (188.0, 76.2)
- added U2: MCP6004, FSFootprints:PDIP14_300MC_MCH, F.Cu at (228.1, 75.7)
- moved R6 81.3 mm to (218.4, 50.8)
- moved R1 19.3 mm to (212.9, 85.4), turned to -90 degrees
- moved R4 8.18 mm to (216.9, 90.4), turned to -90 degrees
- moved R3 7.28 mm to (216.9, 85.3), turned to -90 degrees
- moved R2 5.09 mm to (212.9, 90.4), turned to -90 degrees
Connections:
- net Net-(STM-32_Microcontroller1A-PA0) renamed /OUT2*
- net Net-(STM-32_Microcontroller1A-PA1) renamed /OUT1*
- P1 pad D8: unconnected-(P1-PadD8) -> +12V
- P1 pad D9: unconnected-(P1-PadD9) -> GND
Routing:
- net GND: track 386.9 -> 357.9 mm
- net /OUT2*: track 0.00 -> 3.10 mm
- net /Brake Sensor*: track 0.00 -> 3.08 mm
- net /OUT1*: track 0.00 -> 3.06 mm

Commit message: more pcb edits(for my wonderful electrical wizard friend dustin!!!!)
Parts:
- removed R6: 10 ohm, Resistor_SMD:R_0805_2012Metric_Pad1.20x1.40mm_HandSolder
- added FS-2 APPS/ETC Board: LOGO, 1FS_2_Global_Footprint_Library:FORMULA SLUG, F.Cu at (231.8, 54.6)
- moved R3 6.39 mm to (212.7, 90.2)
- moved R1 6.39 mm to (208.7, 90.2)
- moved R2 6.39 mm to (208.7, 95.3)
- moved R4 6.39 mm to (212.7, 95.3)
- moved R7 6.39 mm to (217.3, 90.2)
- moved R8 6.39 mm to (217.3, 95.3)
Connections:
- U1 pad CN3_6: /LED -> unconnected-(U1A-PB0-PadCN3_6)
Routing:
- net /OUT1: track 0.00 -> 90.0 mm, vias 0 -> 1
- net +9V: track 5.31 -> 85.0 mm, vias 0 -> 4
- net /OUT2: track 0.00 -> 76.5 mm
- net /Brake Sensor: track 0.00 -> 50.7 mm
- net GND: track 357.9 -> 398.7 mm, vias 2 -> 3
- net Net-(U2C-+): track 0.00 -> 38.9 mm, vias 0 -> 2
- net Net-(U2A-+): track 0.00 -> 35.4 mm
- net +5V: track 120.3 -> 155.7 mm, vias 0 -> 6
- net /Brake Sensor*: track 3.08 -> 30.7 mm, vias 0 -> 1
- net Net-(U2B-+): track 0.00 -> 26.1 mm
- net /OUT2*: track 3.10 -> 22.2 mm, vias 0 -> 1
- net /OUT1*: track 3.06 -> 19.2 mm
- net +12V: track 56.6 -> 64.7 mm
Other:
- board text added: "FS-2 APPS/ETC Board Formula Slug V 1.1"
