File: APPS_ETCA/APPS_ETC.kicad_sch (KiCad schematic)
At the start: 21 parts, among them P1 DTM1312PC12PDR008, U1 NUCLEO-L432KC, U2 MCP6004, U6 LM7805_TO220, U8 LM7809_TO220

Commit message: pcb debugged
Parts:
- removed R6: 10 ohm, Resistor_SMD:R_0805_2012Metric_Pad1.20x1.40mm_HandSolder, symbol Device:R
Connections:
- net +5V: now also C4.1
- net CANH: no longer C4.1
- net CANL: no longer C4.2
- net GND: now also C4.2
- net LED: no longer U1.CN3_6 (PB0)
Changed lines of the file:
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@@
   (junction (at 139.7 114.3) (diameter 0) (color 0 0 0 0)
   )
-  (junction (at 124.46 25.4) (diameter 0) (color 0 0 0 0)
+  (junction (at 118.11 33.02) (diameter 0) (color 0 0 0 0)
   )
   (junction (at 58.42 44.45) (diameter 0) (color 0 0 0 0)
@@
   (junction (at 177.8 76.2) (diameter 0) (color 0 0 0 0)
   )
-  (junction (at 124.46 33.02) (diameter 0) (color 0 0 0 0)
-  )
   (junction (at 73.66 34.29) (diameter 0) (color 0 0 0 0)
   )
@@
   (junction (at 46.99 91.44) (diameter 0) (color 0 0 0 0)
   )
+  (junction (at 118.11 25.4) (diameter 0) (color 0 0 0 0)
+  )
   (junction (at 148.59 104.14) (diameter 0) (color 0 0 0 0)
   )
@@
     (stroke (width 0) (type default))
   )
+  (wire (pts (xy 118.11 20.32) (xy 118.11 25.4))
+    (stroke (width 0) (type default))
+  )
+  (wire (pts (xy 140.97 21.59) (xy 140.97 25.4))
+    (stroke (width 0) (type default))
+  )
+  (wire (pts (xy 118.11 33.02) (xy 129.54 33.02))
+    (stroke (width 0) (type default))
+  )
   (wire (pts (xy 148.59 110.49) (xy 163.83 110.49))
     (stroke (width 0) (type default))
   )
-  (wire (pts (xy 120.65 27.94) (xy 120.65 25.4))
-    (stroke (width 0) (type default))
-  )
-  (wire (pts (xy 120.65 25.4) (xy 124.46 25.4))
+  (wire (pts (xy 120.65 27.94) (xy 120.65 21.59))
+    (stroke (width 0) (type default))
+  )
+  (wire (pts (xy 120.65 21.59) (xy 140.97 21.59))
     (stroke (width 0) (type default))
   )
@@
     (stroke (width 0) (type default))
   )
-  (wire (pts (xy 88.9 110.49) (xy 96.52 110.49))
-    (stroke (width 0) (type default))
-  )
   (wire (pts (xy 38.1 99.06) (xy 38.1 102.87))
     (stroke (width 0) (type default))
@@
     (stroke (width 0) (type default))
   )
-  (wire (pts (xy 124.46 33.02) (xy 140.97 33.02))
+  (wire (pts (xy 120.65 36.83) (xy 140.97 36.83))
     (stroke (width 0) (type default))
   )
@@
     (stroke (width 0) (type default))
   )
-  (wire (pts (xy 120.65 33.02) (xy 124.46 33.02))
-    (stroke (width 0) (type default))
-  )
   (wire (pts (xy 58.42 36.83) (xy 58.42 39.37))
     (stroke (width 0) (type default))
@@
     (stroke (width 0) (type default))
   )
+  (wire (pts (xy 118.11 25.4) (xy 129.54 25.4))
+    (stroke (width 0) (type default))
+  )
   (wire (pts (xy 24.13 66.04) (xy 43.18 66.04))
     (stroke (width 0) (type default))
@@
     (stroke (width 0) (type default))
   )
+  (wire (pts (xy 140.97 36.83) (xy 140.97 33.02))
+    (stroke (width 0) (type default))
+  )
   (wire (pts (xy 58.42 44.45) (xy 58.42 58.42))
     (stroke (width 0) (type default))
@@
     (stroke (width 0) (type default))
   )
-  (wire (pts (xy 69.85 110.49) (xy 73.66 110.49))
-    (stroke (width 0) (type default))
-  )
   (wire (pts (xy 109.22 90.17) (xy 115.57 90.17))
     (stroke (width 0) (type default))
@@
     (stroke (width 0) (type default))
   )
+  (wire (pts (xy 118.11 25.4) (xy 114.3 25.4))
+    (stroke (width 0) (type default))
+  )
+  (wire (pts (xy 118.11 33.02) (xy 114.3 33.02))
+    (stroke (width 0) (type default))
+  )
   (wire (pts (xy 73.66 34.29) (xy 93.98 34.29))
     (stroke (width 0) (type default))
   )
-  (wire (pts (xy 120.65 30.48) (xy 120.65 33.02))
+  (wire (pts (xy 120.65 30.48) (xy 120.65 36.83))
     (stroke (width 0) (type default))
   )
@@
     (stroke (width 0) (type default))
   )
+  (wire (pts (xy 118.11 38.1) (xy 118.11 33.02))
+    (stroke (width 0) (type default))
+  )
   (wire (pts (xy 73.66 25.4) (xy 73.66 26.67))
     (stroke (width 0) (type default))
   )
-  (wire (pts (xy 78.74 74.93) (xy 68.58 74.93))
-    (stroke (width 0) (type default))
-  )
   (wire (pts (xy 245.11 17.78) (xy 245.11 24.13))
     (stroke (width 0) (type default))
@@
   )
   (wire (pts (xy 109.22 85.09) (xy 123.19 85.09))
-    (stroke (width 0) (type default))
-  )
-  (wire (pts (xy 124.46 25.4) (xy 140.97 25.4))
     (stroke (width 0) (type default))
   )
@@
   )
   (label "OUT1" (at 166.37 63.5 0) (fields_autoplaced)
-    (effects (font (size 1.27 1.27)) (justify left bottom))
-  )
-  (label "LED" (at 69.85 110.49 0) (fields_autoplaced)
     (effects (font (size 1.27 1.27)) (justify left bottom))
   )
@@
         (path "/21da8b0a-bf7f-4003-9579-5de7190091be"
           (reference "#PWR021") (unit 1)
+        )
+      )
+    )
+  )
+  (symbol (lib_id "Device:C") (at 129.54 29.21 0) (unit 1)
+    (in_bom yes) (on_board yes) (dnp no) (fields_autoplaced)
+    (property "Reference" "C4" (at 133.35 27.94 0)
+      (effects (font (size 1.27 1.27)) (justify left))
+    )
+    (property "Value" "100nF" (at 133.35 30.48 0)
+      (effects (font (size 1.27 1.27)) (justify left))
+    )
+    (property "Footprint" "Capacitor_SMD:C_0805_2012Metric_Pad1.18x1.45mm_HandSolder" (at 130.5052 33.02 0)
+      (effects (font (size 1.27 1.27)) hide)
+    )
+    (property "Datasheet" "~" (at 129.54 29.21 0)
+      (effects (font (size 1.27 1.27)) hide)
+    )
+    (pin "1")
+    (pin "2")
+    (instances
+      (project "APPS_ETC"
+        (path "/21da8b0a-bf7f-4003-9579-5de7190091be"
+          (reference "C4") (unit 1)
         )
       )
@@
     )
   )
-  (symbol (lib_id "power:GND") (at 114.3 33.02 90) (unit 1)
-    (in_bom yes) (on_board yes) (dnp no) (fields_autoplaced)
-    (property "Reference" "#PWR020" (at 120.65 33.02 0)
-      (effects (font (size 1.27 1.27)) hide)
-    )
-    (property "Value" "GND" (at 118.11 33.02 90)
-      (effects (font (size 1.27 1.27)) (justify right))
-    )
-    (property "Footprint" "" (at 114.3 33.02 0)
-      (effects (font (size 1.27 1.27)) hide)
-    )
-    (property "Datasheet" "" (at 114.3 33.02 0)
+  (symbol (lib_id "power:GND") (at 118.11 38.1 0) (unit 1)
+    (in_bom yes) (on_board yes) (dnp no) (fields_autoplaced)
+    (property "Reference" "#PWR020" (at 118.11 44.45 0)
+      (effects (font (size 1.27 1.27)) hide)
+    )
+    (property "Value" "GND" (at 120.65 39.37 0)
+      (effects (font (size 1.27 1.27)) (justify left))
+    )
+    (property "Footprint" "" (at 118.11 38.1 0)
+      (effects (font (size 1.27 1.27)) hide)
+    )
+    (property "Datasheet" "" (at 118.11 38.1 0)
       (effects (font (size 1.27 1.27)) hide)
     )
@@
     )
   )
-  (symbol (lib_id "Device:R") (at 77.47 110.49 270) (unit 1)
-    (in_bom yes) (on_board yes) (dnp no) (fields_autoplaced)
-    (property "Reference" "R6" (at 77.47 104.14 90)
-      (effects (font (size 1.27 1.27)))
-    )
-    (property "Value" "10 ohm" (at 77.47 106.68 90)
-      (effects (font (size 1.27 1.27)))
-    )
-    (property "Footprint" "Resistor_SMD:R_0805_2012Metric_Pad1.20x1.40mm_HandSolder" (at 77.47 108.712 90)
-      (effects (font (size 1.27 1.27)) hide)
-    )
-    (property "Datasheet" "~" (at 77.47 110.49 0)
-      (effects (font (size 1.27 1.27)) hide)
-    )
-    (pin "1")
-    (pin "2")
-    (instances
-      (project "APPS_ETC"
-        (path "/21da8b0a-bf7f-4003-9579-5de7190091be"
-          (reference "R6") (unit 1)
-        )
-      )
-    )
-  )
   (symbol (lib_id "power:+12V") (at 43.18 66.04 0) (unit 1)
     (in_bom yes) (on_board yes) (dnp no) (fields_autoplaced)
@@
         (path "/21da8b0a-bf7f-4003-9579-5de7190091be"
           (reference "#PWR025") (unit 1)
-        )
-      )
-    )
-  )
-  (symbol (lib_id "Device:C") (at 124.46 29.21 0) (unit 1)
-    (in_bom yes) (on_board yes) (dnp no) (fields_autoplaced)
-    (property "Reference" "C4" (at 128.27 27.94 0)
-      (effects (font (size 1.27 1.27)) (justify left))
-    )
-    (property "Value" "100nF" (at 128.27 30.48 0)
-      (effects (font (size 1.27 1.27)) (justify left))
-    )
-    (property "Footprint" "Capacitor_SMD:C_0805_2012Metric_Pad1.18x1.45mm_HandSolder" (at 125.4252 33.02 0)
-      (effects (font (size 1.27 1.27)) hide)
-    )
-    (property "Datasheet" "~" (at 124.46 29.21 0)
-      (effects (font (size 1.27 1.27)) hide)
-    )
-    (pin "1")
-    (pin "2")
-    (instances
-      (project "APPS_ETC"
-        (path "/21da8b0a-bf7f-4003-9579-5de7190091be"
-          (reference "C4") (unit 1)
         )
       )
@@
     )
   )
-  (symbol (lib_id "power:+5V") (at 114.3 25.4 0) (unit 1)
-    (in_bom yes) (on_board yes) (dnp no) (fields_autoplaced)
-    (property "Reference" "#PWR02" (at 114.3 29.21 0)
-      (effects (font (size 1.27 1.27)) hide)
-    )
-    (property "Value" "+5V" (at 114.3 20.32 0)
-      (effects (font (size 1.27 1.27)))
-    )
-    (property "Footprint" "" (at 114.3 25.4 0)
-      (effects (font (size 1.27 1.27)) hide)
-    )
-    (property "Datasheet" "" (at 114.3 25.4 0)
+  (symbol (lib_id "power:+5V") (at 118.11 20.32 0) (unit 1)
+    (in_bom yes) (on_board yes) (dnp no) (fields_autoplaced)
+    (property "Reference" "#PWR02" (at 118.11 24.13 0)
+      (effects (font (size 1.27 1.27)) hide)
+    )
+    (property "Value" "+5V" (at 118.11 15.24 0)
+      (effects (font (size 1.27 1.27)))
+    )
+    (property "Footprint" "" (at 118.11 20.32 0)
+      (effects (font (size 1.27 1.27)) hide)
+    )
+    (property "Datasheet" "" (at 118.11 20.32 0)
       (effects (font (size 1.27 1.27)) hide)
     )
@@
         )
       )
-    )
-  )
-  (symbol (lib_id "power:GND") (at 96.52 110.49 0) (unit 1)
-    (in_bom yes) (on_board yes) (dnp no) (fields_autoplaced)
-    (property "Reference" "#PWR027" (at 96.52 116.84 0)
-      (effects (font (size 1.27 1.27)) hide)
-    )
-    (property "Value" "GND" (at 96.52 115.57 0)
-      (effects (font (size 1.27 1.27)))
-    )
-    (property "Footprint" "" (at 96.52 110.49 0)
-      (effects (font (size 1.27 1.27)) hide)
-    )
-    (property "Datasheet" "" (at 96.52 110.49 0)
-      (effects (font (size 1.27 1.27)) hide)
-    )
-    (pin "1")
-    (instances
-      (project "APPS_ETC"
-        (path "/21da8b0a-bf7f-4003-9579-5de7190091be"
-          (reference "#PWR027") (unit 1)
-        )
-      )

Commit message: pcb done!!!
Parts:
- R4: value 330kO -> 180kO
Other:
- moved on the sheet: C3
Changed lines of the file:
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@@
   (junction (at 177.8 76.2) (diameter 0) (color 0 0 0 0)
   )
-  (junction (at 73.66 34.29) (diameter 0) (color 0 0 0 0)
-  )
   (junction (at 26.67 91.44) (diameter 0) (color 0 0 0 0)
   )
@@
   (junction (at 118.11 25.4) (diameter 0) (color 0 0 0 0)
   )
+  (junction (at 73.66 33.02) (diameter 0) (color 0 0 0 0)
+  )
   (junction (at 148.59 104.14) (diameter 0) (color 0 0 0 0)
   )
@@
     (stroke (width 0) (type default))
   )
+  (wire (pts (xy 73.66 33.02) (xy 73.66 38.1))
+    (stroke (width 0) (type default))
+  )
   (wire (pts (xy 181.61 66.04) (xy 182.88 66.04))
     (stroke (width 0) (type default))
@@
     (stroke (width 0) (type default))
   )
-  (wire (pts (xy 73.66 34.29) (xy 73.66 38.1))
-    (stroke (width 0) (type default))
-  )
   (wire (pts (xy 160.02 63.5) (xy 166.37 63.5))
     (stroke (width 0) (type default))
@@
     (stroke (width 0) (type default))
   )
+  (wire (pts (xy 73.66 22.86) (xy 73.66 25.4))
+    (stroke (width 0) (type default))
+  )
   (wire (pts (xy 118.11 25.4) (xy 114.3 25.4))
     (stroke (width 0) (type default))
@@
     (stroke (width 0) (type default))
   )
-  (wire (pts (xy 73.66 34.29) (xy 93.98 34.29))
+  (wire (pts (xy 73.66 33.02) (xy 93.98 33.02))
     (stroke (width 0) (type default))
   )
@@
     (stroke (width 0) (type default))
   )
-  (wire (pts (xy 93.98 34.29) (xy 93.98 33.02))
-    (stroke (width 0) (type default))
-  )
   (wire (pts (xy 118.11 38.1) (xy 118.11 33.02))
-    (stroke (width 0) (type default))
-  )
-  (wire (pts (xy 73.66 25.4) (xy 73.66 26.67))
     (stroke (width 0) (type default))
   )
@@
   (text "MCU\n" (at 111.76 116.84 0)
     (effects (font (size 2 2)) (justify left bottom))
-  )
-  (label "LED" (at 68.58 74.93 0) (fields_autoplaced)
-    (effects (font (size 1.27 1.27)) (justify left bottom))
   )
   (label "OUT2" (at 260.35 62.23 90) (fields_autoplaced)
@@
     )
   )
-  (symbol (lib_id "Device:C") (at 73.66 30.48 0) (unit 1)
-    (in_bom yes) (on_board yes) (dnp no) (fields_autoplaced)
-    (property "Reference" "C3" (at 77.47 29.21 0)
-      (effects (font (size 1.27 1.27)) (justify left))
-    )
-    (property "Value" "100nF" (at 77.47 31.75 0)
-      (effects (font (size 1.27 1.27)) (justify left))
-    )
-    (property "Footprint" "Capacitor_SMD:C_0805_2012Metric_Pad1.18x1.45mm_HandSolder" (at 74.6252 34.29 0)
-      (effects (font (size 1.27 1.27)) hide)
-    )
-    (property "Datasheet" "~" (at 73.66 30.48 0)
+  (symbol (lib_id "Device:C") (at 73.66 29.21 0) (unit 1)
+    (in_bom yes) (on_board yes) (dnp no) (fields_autoplaced)
+    (property "Reference" "C3" (at 77.47 27.94 0)
+      (effects (font (size 1.27 1.27)) (justify left))
+    )
+    (property "Value" "100nF" (at 77.47 30.48 0)
+      (effects (font (size 1.27 1.27)) (justify left))
+    )
+    (property "Footprint" "Capacitor_SMD:C_0805_2012Metric_Pad1.18x1.45mm_HandSolder" (at 74.6252 33.02 0)
+      (effects (font (size 1.27 1.27)) hide)
+    )
+    (property "Datasheet" "~" (at 73.66 29.21 0)
       (effects (font (size 1.27 1.27)) hide)
     )
@@
       (effects (font (size 1.27 1.27)) (justify left))
     )
-    (property "Value" "330kO" (at 142.24 120.65 0)
+    (property "Value" "180kO" (at 142.24 120.65 0)
       (effects (font (size 1.27 1.27)) (justify left))
     )
@@
     )
   )
-  (symbol (lib_id "power:+3.3V") (at 73.66 25.4 0) (unit 1)
-    (in_bom yes) (on_board yes) (dnp no) (fields_autoplaced)
-    (property "Reference" "#PWR06" (at 73.66 29.21 0)
-      (effects (font (size 1.27 1.27)) hide)
-    )
-    (property "Value" "+3.3V" (at 73.66 20.32 0)
-      (effects (font (size 1.27 1.27)))
-    )
-    (property "Footprint" "" (at 73.66 25.4 0)
-      (effects (font (size 1.27 1.27)) hide)
-    )
-    (property "Datasheet" "" (at 73.66 25.4 0)
-      (effects (font (size 1.27 1.27)) hide)
-    )
+  (symbol (lib_id "power:+3.3V") (at 73.66 22.86 0) (unit 1)
+    (in_bom yes) (on_board yes) (dnp no) (fields_autoplaced)
+    (property "Reference" "#PWR06" (at 73.66 26.67 0)
+      (effects (font (size 1.27 1.27)) hide)
+    )
+    (property "Value" "+3.3V" (at 73.66 17.78 0)
+      (effects (font (size 1.27 1.27)))
+    )
+    (property "Footprint" "" (at 73.66 22.86 0)
+      (effects (font (size 1.27 1.27)) hide)
+    )
+    (property "Datasheet" "" (at 73.66 22.86 0)
+      (effects (font (size 1.27 1.27)) hide)
+    )

Commit message: updated pcb
Connections:
- net Brake Sensor: now also U2.10 (+); no longer U2.9 (-)
- net OUT1: now also U2.3 (+); no longer U2.2 (-)
- net OUT2: now also U2.5 (+); no longer U2.6 (-)
- net at R7.1, U2.8: now also U2.9 (-); no longer U2.10 (+)
- net at R3.1, U2.7: now also U2.6 (-); no longer U2.5 (+)
- net at R1.1, U2.1: now also U2.2 (-); no longer U2.3 (+)
Other:
- moved on the sheet: U2A, U2B, U2C
Changed lines of the file:
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@@
     )
   )
-  (symbol (lib_id "Amplifier_Operational:MCP6004") (at 190.5 66.04 180) (unit 3)
-    (in_bom yes) (on_board yes) (dnp no) (fields_autoplaced)
-    (property "Reference" "U2" (at 190.5 55.88 0)
-      (effects (font (size 1.27 1.27)))
-    )
-    (property "Value" "MCP6004" (at 190.5 58.42 0)
-      (effects (font (size 1.27 1.27)))
-    )
-    (property "Footprint" "FSFootprints:PDIP14_300MC_MCH" (at 191.77 68.58 0)
-      (effects (font (size 1.27 1.27)) hide)
-    )
-    (property "Datasheet" "http://ww1.microchip.com/downloads/en/DeviceDoc/21733j.pdf" (at 189.23 71.12 0)
+  (symbol (lib_id "Amplifier_Operational:MCP6004") (at 190.5 66.04 0) (mirror y) (unit 3)
+    (in_bom yes) (on_board yes) (dnp no)
+    (property "Reference" "U2" (at 190.5 76.2 0)
+      (effects (font (size 1.27 1.27)))
+    )
+    (property "Value" "MCP6004" (at 190.5 73.66 0)
+      (effects (font (size 1.27 1.27)))
+    )
+    (property "Footprint" "FSFootprints:PDIP14_300MC_MCH" (at 191.77 63.5 0)
+      (effects (font (size 1.27 1.27)) hide)
+    )
+    (property "Datasheet" "http://ww1.microchip.com/downloads/en/DeviceDoc/21733j.pdf" (at 189.23 60.96 0)
       (effects (font (size 1.27 1.27)) hide)
     )
@@
     )
   )
-  (symbol (lib_id "Amplifier_Operational:MCP6004") (at 152.4 66.04 180) (unit 1)
-    (in_bom yes) (on_board yes) (dnp no) (fields_autoplaced)
-    (property "Reference" "U2" (at 152.4 55.88 0)
-      (effects (font (size 1.27 1.27)))
-    )
-    (property "Value" "MCP6004" (at 152.4 58.42 0)
-      (effects (font (size 1.27 1.27)))
-    )
-    (property "Footprint" "FSFootprints:PDIP14_300MC_MCH" (at 153.67 68.58 0)
-      (effects (font (size 1.27 1.27)) hide)
-    )
-    (property "Datasheet" "http://ww1.microchip.com/downloads/en/DeviceDoc/21733j.pdf" (at 151.13 71.12 0)
+  (symbol (lib_id "Amplifier_Operational:MCP6004") (at 152.4 66.04 0) (mirror y) (unit 1)
+    (in_bom yes) (on_board yes) (dnp no)
+    (property "Reference" "U2" (at 152.4 76.2 0)
+      (effects (font (size 1.27 1.27)))
+    )
+    (property "Value" "MCP6004" (at 152.4 73.66 0)
+      (effects (font (size 1.27 1.27)))
+    )
+    (property "Footprint" "FSFootprints:PDIP14_300MC_MCH" (at 153.67 63.5 0)
+      (effects (font (size 1.27 1.27)) hide)
+    )
+    (property "Datasheet" "http://ww1.microchip.com/downloads/en/DeviceDoc/21733j.pdf" (at 151.13 60.96 0)
       (effects (font (size 1.27 1.27)) hide)
     )
@@
     )
   )
-  (symbol (lib_id "Amplifier_Operational:MCP6004") (at 156.21 104.14 180) (unit 2)
-    (in_bom yes) (on_board yes) (dnp no) (fields_autoplaced)
-    (property "Reference" "U2" (at 156.21 93.98 0)
-      (effects (font (size 1.27 1.27)))
-    )
-    (property "Value" "MCP6004" (at 156.21 96.52 0)
-      (effects (font (size 1.27 1.27)))
-    )
-    (property "Footprint" "FSFootprints:PDIP14_300MC_MCH" (at 157.48 106.68 0)
-      (effects (font (size 1.27 1.27)) hide)
-    )
-    (property "Datasheet" "http://ww1.microchip.com/downloads/en/DeviceDoc/21733j.pdf" (at 154.94 109.22 0)
-      (effects (font (size 1.27 1.27)) hide)
-    )
+  (symbol (lib_id "Amplifier_Operational:MCP6004") (at 156.21 104.14 0) (mirror y) (unit 2)
+    (in_bom yes) (on_board yes) (dnp no)
+    (property "Reference" "U2" (at 156.21 114.3 0)
+      (effects (font (size 1.27 1.27)))
+    )
+    (property "Value" "MCP6004" (at 156.21 111.76 0)
+      (effects (font (size 1.27 1.27)))
+    )
+    (property "Footprint" "FSFootprints:PDIP14_300MC_MCH" (at 157.48 101.6 0)
+      (effects (font (size 1.27 1.27)) hide)
+    )
+    (property "Datasheet" "http://ww1.microchip.com/downloads/en/DeviceDoc/21733j.pdf" (at 154.94 99.06 0)
+      (effects (font (size 1.27 1.27)) hide)
+    )
