File: APPS_ETCA/_autosave-APPS_ETC.kicad_pcb (KiCad board)
At the start: 2 copper layers, 81.3 x 99.1 mm, 20 parts, among them P1 DTM1312PC12PDR008, U1 NUCLEO-L432KC, U2 MCP6004, U6 LM7805_TO220, U8 LM7809_TO220

Commit message: PCB - prototype done
Parts:
- added FS-2 APPS/ETC Board: LOGO, 1FS_2_Global_Footprint_Library:FORMULA SLUG, F.Cu at (224.8, 52.1)
Other:
- board text added: "FS-2 APPS/ETC Board Formula Slug V 1.1"
