File: Charging Shutdown Circuit/Charging Shutdown Circuit.kicad_pcb (KiCad board)
At the start: 2 copper layers, 9 parts, among them K2 ALDP112W, K3 ALDP112W, K4 GIGAVAC GX14BB, K5 GIGAVAC GX14BB, SW1 SW-STOP, SW2 SW_HVD_IL, U1 AQY2805X, U2 AQY2805X

Commit message: charger stuff (don't break plz)
Parts:
- added C1: 1uf, Capacitor_SMD:C_0805_2012Metric_Pad1.18x1.45mm_HandSolder, F.Cu at (80.4, 78.1)
- added C2: 100nf, Capacitor_SMD:C_0805_2012Metric_Pad1.18x1.45mm_HandSolder, F.Cu at (80.4, 81.1)
- added D1: D, Diode_SMD:D_2010_5025Metric_Pad1.52x2.65mm_HandSolder, F.Cu at (63.3, 67.0)
- added D2: D, Diode_SMD:D_2010_5025Metric_Pad1.52x2.65mm_HandSolder, F.Cu at (63.3, 71.3)
- added D3: D, Diode_SMD:D_2010_5025Metric_Pad1.52x2.65mm_HandSolder, F.Cu at (63.3, 75.5)
- added D4: D, Diode_SMD:D_2010_5025Metric_Pad1.52x2.65mm_HandSolder, F.Cu at (63.3, 79.8)
- added D5: D, Diode_SMD:D_2010_5025Metric_Pad1.52x2.65mm_HandSolder, F.Cu at (63.3, 84.1)
- added J1: IMD, 1FS_2_Global_Footprint_Library:MOLEX_1053091203, F.Cu at (82.8, 49.3)
- added J2: Shutdown IL, 1FS_2_Global_Footprint_Library:MOLEX_1053091202, F.Cu at (82.8, 39.4)
- added J4: 776087-1, 1FS_2_Global_Footprint_Library:TE_776087-1, F.Cu at (23.0, 33.0)
- added K1: Latching Relay, 1FS_2_Global_Footprint_Library:Omron G6BK-1114P-US, F.Cu at (84.6, 22.7)
- added Q1: STS6NF20V, 1FS_2_Global_Footprint_Library:SO-8_STM, F.Cu at (89.0, 59.1)
- added R1: 1600, Resistor_SMD:R_0805_2012Metric_Pad1.20x1.40mm_HandSolder, F.Cu at (91.2, -13.1)
- added R2: 560, Resistor_SMD:R_0805_2012Metric_Pad1.20x1.40mm_HandSolder, F.Cu at (91.2, -10.1)
- added R3: 665, Resistor_SMD:R_0805_2012Metric_Pad1.20x1.40mm_HandSolder, F.Cu at (91.2, -7.15)
- added R4: 370, Resistor_SMD:R_0805_2012Metric_Pad1.20x1.40mm_HandSolder, F.Cu at (91.2, -4.20)
- added R5: 205, Resistor_SMD:R_0805_2012Metric_Pad1.20x1.40mm_HandSolder, F.Cu at (91.2, -1.25)
- added R6: 370, Resistor_SMD:R_0805_2012Metric_Pad1.20x1.40mm_HandSolder, F.Cu at (91.2, 1.70)
- added R7: 374, Resistor_SMD:R_0805_2012Metric_Pad1.20x1.40mm_HandSolder, F.Cu at (91.2, 4.65)
- added R8: 2.4M, Resistor_SMD:R_0805_2012Metric_Pad1.20x1.40mm_HandSolder, F.Cu at (91.2, 7.60)
- added SW2: SH_RESET, Button_Switch_SMD:Nidec_Copal_CAS-120A, F.Cu at (82.0, 59.2)
- added U1: DK1A1B-12V, 1FS_2_Global_Footprint_Library:RELAY_DK2A_PAN, F.Cu at (17.8, 67.3)
- added U10: NAND, Package_DIP:DIP-14_W7.62mm, F.Cu at (68.8, 66.9)
- added U11: LM555N, Package_DIP:DIP-8_W7.62mm, F.Cu at (79.6, 66.9)
- added U3: NSL-32, 1FS_2_Global_Footprint_Library:OptoCoupler 6-SOP, F.Cu at (84.0, -11.8)
- added U4: NSL-32, 1FS_2_Global_Footprint_Library:OptoCoupler 6-SOP, F.Cu at (84.0, -6.48)
- added U5: DK1A1B-12V, 1FS_2_Global_Footprint_Library:RELAY_DK2A_PAN, F.Cu at (33.0, 66.8)
- added U6: NSL-32, 1FS_2_Global_Footprint_Library:OptoCoupler 6-SOP, F.Cu at (84.0, -1.11)
- added U7: NSL-32, 1FS_2_Global_Footprint_Library:OptoCoupler 6-SOP, F.Cu at (84.0, 4.26)
- added U8: DK1A1B-12V, 1FS_2_Global_Footprint_Library:RELAY_DK2A_PAN, F.Cu at (47.2, 66.8)
- added U9: NSL-32, 1FS_2_Global_Footprint_Library:OptoCoupler 6-SOP, F.Cu at (84.0, 9.63)
- moved K5 3.81 mm to (158.9, 53.7)
Connections:
- SW1 pad 1: Net-(SW1-A) -> /Shutdown_ACC_IN
- SW1 pad 2: Net-(SW1-B) -> +12V
Routing:
- net GND: track 0.00 -> 24.4 mm
Other:
- board outline added: 139.7 x 88.9 mm
