File: Charging Shutdown Circuit/Charging Shutdown Circuit.kicad_sch (KiCad schematic)
At the start: 36 parts, among them J1 IMD, J2 Shutdown IL, J3 776087-1, J4 776087-1, K1 Latching Relay, K4 GIGAVAC GX14BAB, K5 GIGAVAC GX14BB, Q1 STS6NF20V, SW1 SW-STOP, SW2 SH_RESET, U1 DK1A1B-12V, U10 NAND, U11 LM555N, U3 NSL-32, U4 NSL-32, U5 DK1A1B-12V, U6 NSL-32, U7 NSL-32, U8 DK1A1B-12V, U9 NSL-32

Commit message: charging changes duhhh
Parts:
- added R10: 6.8k, symbol Device:R
- added R9: 18k, symbol Device:R
Connections:
- net Shutdown_AIRS_IN is gone; now on net Shutdown_ACC_OUT: J3.20, J4.20
- net +12V: now also R9.1
- net Charge_State: now also R10.1, R9.2
- net GND: now also R10.2
Changed lines of the file:
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@@
   (junction (at 238.76 256.54) (diameter 0) (color 0 0 0 0)
+  )
+  (junction (at 436.88 255.27) (diameter 0) (color 0 0 0 0)
   )
   (junction (at 35.56 254) (diameter 0) (color 0 0 0 0)
@@
     (stroke (width 0) (type default))
   )
+  (wire (pts (xy 556.26 196.85) (xy 485.14 196.85))
+    (stroke (width 0) (type default))
+  )
   (wire (pts (xy 35.56 236.22) (xy 35.56 245.11))
     (stroke (width 0) (type default))
@@
     (stroke (width 0) (type default))
   )
+  (wire (pts (xy 425.45 254) (xy 425.45 255.27))
+    (stroke (width 0) (type default))
+  )
   (wire (pts (xy 502.92 321.31) (xy 574.04 321.31))
     (stroke (width 0) (type default))
@@
     (stroke (width 0) (type default))
   )
+  (wire (pts (xy 436.88 255.27) (xy 436.88 260.35))
+    (stroke (width 0) (type default))
+  )
   (wire (pts (xy 62.23 326.39) (xy 77.47 326.39))
     (stroke (width 0) (type default))
@@
     (stroke (width 0) (type default))
   )
+  (wire (pts (xy 485.14 196.85) (xy 485.14 190.5))
+    (stroke (width 0) (type default))
+  )
   (wire (pts (xy 176.53 256.54) (xy 180.34 256.54))
     (stroke (width 0) (type default))
@@
     (stroke (width 0) (type default))
   )
+  (wire (pts (xy 425.45 255.27) (xy 429.26 255.27))
+    (stroke (width 0) (type default))
+  )
   (wire (pts (xy 485.14 190.5) (xy 520.7 190.5))
     (stroke (width 0) (type default))
   )
+  (wire (pts (xy 556.26 190.5) (xy 556.26 196.85))
+    (stroke (width 0) (type default))
+  )
   (wire (pts (xy 238.76 256.54) (xy 238.76 254))
     (stroke (width 0) (type default))
@@
   )
   (wire (pts (xy 466.09 281.94) (xy 487.68 281.94))
+    (stroke (width 0) (type default))
+  )
+  (wire (pts (xy 444.5 255.27) (xy 453.39 255.27))
     (stroke (width 0) (type default))
   )
@@
   (label "IMD_FAULT_5V" (at 77.47 326.39 180) (fields_autoplaced)
     (effects (font (size 1.27 1.27)) (justify right bottom))
+  )
+  (label "Charge_State" (at 436.88 260.35 0) (fields_autoplaced)
+    (effects (font (size 1.27 1.27)) (justify left bottom))
   )
   (label "SH_RESET" (at 471.17 321.31 0) (fields_autoplaced)
@@
     )
   )
+  (symbol (lib_id "power:+12V") (at 425.45 254 0) (unit 1)
+    (in_bom yes) (on_board yes) (dnp no) (fields_autoplaced)
+    (property "Reference" "#PWR036" (at 425.45 257.81 0)
+      (effects (font (size 1.27 1.27)) hide)
+    )
+    (property "Value" "+12V" (at 425.45 248.92 0)
+      (effects (font (size 1.27 1.27)))
+    )
+    (property "Footprint" "" (at 425.45 254 0)
+      (effects (font (size 1.27 1.27)) hide)
+    )
+    (property "Datasheet" "" (at 425.45 254 0)
+      (effects (font (size 1.27 1.27)) hide)
+    )
+    (pin "1")
+    (instances
+      (project "Charging Shutdown Circuit"
+        (path "/160379ad-6194-4298-b157-948e3cc7f004"
+          (reference "#PWR036") (unit 1)
+        )
+      )
+    )
+  )
   (symbol (lib_name "R_1") (lib_id "Device:R") (at 90.17 247.65 90) (unit 1)
     (in_bom yes) (on_board yes) (dnp no)
@@
         (path "/e19d26dd-723b-45e6-9d59-b1730158e759"
           (reference "K2") (unit 1)
+        )
+      )
+    )
+  )
+  (symbol (lib_id "Device:R") (at 440.69 255.27 90) (unit 1)
+    (in_bom yes) (on_board yes) (dnp no) (fields_autoplaced)
+    (property "Reference" "R10" (at 440.69 248.92 90)
+      (effects (font (size 1.27 1.27)))
+    )
+    (property "Value" "6.8k" (at 440.69 251.46 90)
+      (effects (font (size 1.27 1.27)))
+    )
+    (property "Footprint" "" (at 440.69 257.048 90)
+      (effects (font (size 1.27 1.27)) hide)
+    )
+    (property "Datasheet" "~" (at 440.69 255.27 0)
+      (effects (font (size 1.27 1.27)) hide)
+    )
+    (pin "1")
+    (pin "2")
+    (instances
+      (project "Charging Shutdown Circuit"
+        (path "/160379ad-6194-4298-b157-948e3cc7f004"
+          (reference "R10") (unit 1)
         )
       )
@@
     )
   )
+  (symbol (lib_id "power:GND") (at 453.39 255.27 0) (unit 1)
+    (in_bom yes) (on_board yes) (dnp no) (fields_autoplaced)
+    (property "Reference" "#PWR037" (at 453.39 261.62 0)
+      (effects (font (size 1.27 1.27)) hide)
+    )
+    (property "Value" "GND" (at 453.39 260.35 0)
+      (effects (font (size 1.27 1.27)))
+    )
+    (property "Footprint" "" (at 453.39 255.27 0)
+      (effects (font (size 1.27 1.27)) hide)
+    )
+    (property "Datasheet" "" (at 453.39 255.27 0)
+      (effects (font (size 1.27 1.27)) hide)
+    )
+    (pin "1")
+    (instances
+      (project "Charging Shutdown Circuit"
+        (path "/160379ad-6194-4298-b157-948e3cc7f004"
+          (reference "#PWR037") (unit 1)
+        )
+      )
+    )
+  )
   (symbol (lib_id "2FS-1_Symbol Library:DK1A1B-12V") (at 444.5 321.31 90) (mirror x) (unit 1)
     (in_bom yes) (on_board yes) (dnp no)
@@
         )
       )
+    )
+  )
+  (symbol (lib_id "Device:R") (at 433.07 255.27 90) (unit 1)
+    (in_bom yes) (on_board yes) (dnp no) (fields_autoplaced)
+    (property "Reference" "R9" (at 433.07 248.92 90)
+      (effects (font (size 1.27 1.27)))
+    )
+    (property "Value" "18k" (at 433.07 251.46 90)
+      (effects (font (size 1.27 1.27)))
+    )
+    (property "Footprint" "" (at 433.07 257.048 90)
+      (effects (font (size 1.27 1.27)) hide)
+    )
+    (property "Datasheet" "~" (at 433.07 255.27 0)
+      (effects (font (size 1.27 1.27)) hide)
+    )
+    (pin "1")
+    (pin "2")
+    (instances
+      (project "Charging Shutdown Circuit"
+        (path "/160379ad-6194-4298-b157-948e3cc7f004"
+          (reference "R9") (unit 1)
+        )
+      )

Commit message: charger stuff (don't break plz)
Parts:
- removed U10: NAND, Package_DIP:DIP-14_W7.62mm, symbol 4xxx:4023
- removed U11: LM555N, Package_DIP:DIP-8_W7.62mm, symbol 2FS-1_Symbol Library:LM555N
- removed U3, U4, U6, U7, U9: NSL-32, 1FS_2_Global_Footprint_Library:OptoCoupler 6-SOP, symbol Isolator:NSL-32
- removed U8: DK1A1B-12V, 1FS_2_Global_Footprint_Library:RELAY_DK2A_PAN, symbol 2FS-1_Symbol Library:DK1A1B-12V
- added U10: LM555N, Package_DIP:DIP-8_W7.62mm, symbol 2FS-1_Symbol Library:LM555N
- added U2, U4, U6, U7, U8: TLP3122AE, 1FS_2_Global_Footprint_Library:OptoCoupler 6-SOP, symbol 1FS_2_Global_Symbol_Library:TLP3122AE
- added U3: DK1A1B-12V, 1FS_2_Global_Footprint_Library:RELAY_DK2A_PAN, symbol 2FS-1_Symbol Library:DK1A1B-12V
- added U9: NAND, Package_DIP:DIP-14_W7.62mm, symbol 4xxx:4023
- R7: value 374 -> 370
Connections:
- net +12V: now also D1.1 (K), U3.8 (+), U4.4, U7.4, U8.4
- net +5V: now also U10.4 (R), U10.8 (VCC), U2.4, U6.4, U9.14 (VDD)
- net BMS_FAULT: now also U6.3
- net BMS_FAULT_5V: now also U4.3, U6.6, U9.8
- net GND: now also R3.2, R5.2, U10.1 (GND), U3.1 (-), U4.6, U9.7 (VSS)
- net IMD_FAULT: now also U2.3
- net IMD_FAULT_5V: now also U2.6, U7.3, U9.1, U9.2
- net IMD_Latch_Delay: now also U10.3 (Q)
- net Shutdown_ACC_IN: now also U3.3; no longer U5.3
- net at R6.2: now also U7.1
- net at D2.1 (K): now also U5.8 (+), U7.6
- net at U5.4: now also J2.1
- net at R3.1: now also U2.1
- net at R5.1: now also U6.1
- net at J2.2: now also K1.4
- net at C1.2, R8.1: now also U10.2 (TR), U10.6 (THR)
- net at R7.1: now also U8.1
- net at D3.1 (K), K1.5: now also U8.6
- net at R4.1: now also U4.1
- new net: U3.4, U5.3
- new net: U8.3, U9.9
