File: discharge/tractive/tractive.kicad_sch (KiCad schematic)
At the start: 20 parts, among them J1 TS, J2 CAN, J2 GLV, J2 Shutdown, J3 776261-1, U3 PQDE6W-Q110-S5-H-D

Commit message: Mid Updating Tractive Board to Mesh with Github
Parts:
- removed H1, H2, H3, H4: MountingHole, discharge:hole, symbol Mechanical:MountingHole
- D2: footprint Library:D_DO-41_SOD81_P10.16mm_Horizontal -> Diode_THT:D_DO-41_SOD81_P10.16mm_Horizontal
- J1, J2: footprint Library:MOLEX_1053091202 -> 1FS_2_Global_Footprint_Library:MOLEX_1053091202
- J3: footprint Library:CONN14_776261_TEC -> 1FS_2_Global_Footprint_Library:CONN14_776261_TEC
- PhoenixContact: footprint Library:relay -> 1FS_2_Global_Footprint_Library:PhoenixContact1
- TEConnectivityDT15-2P2: footprint Library:CONN2_DT15-2P_TEC -> 1FS_2_Global_Footprint_Library:TEConnectivityDT15-2P1
Connections:
- net at PhoenixContact.3: now also D2.1 (K), J1.2, R2.1
- net at PhoenixContact.4 (switching): now also R1.1
- net at TEConnectivityDT15-2P2.2: now also R2.2; no longer R2.1
Other:
- moved on the sheet: D2, J1, J2, J3, PhoenixContact, R1, R2, R3, R5, R6, TEConnectivityDT15-2P2, U2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
