File: Telemetry Board/Telemetry Board.kicad_pcb (KiCad board)
At the start: 2 copper layers, 76.2 x 53.3 mm, 18 parts, among them J1 776180-1, U1 LM7805_TO220, U2 LM7809_TO220, U3 CD74HC4067SM96, U4 ISO1050DUB, U5 NUCLEO-L432KC

Commit message: Telemetry Board V1 Done
Parts:
- added G***: LOGO, 1FS_2_Global_Footprint_Library:FS_Logo_4LinesTall, F.Cu at (63.7, 61.9)
- added REF**: MountingHole_3.5mm, MountingHole:MountingHole_3.5mm, F.Cu at (91.9, 94.0)
- added REF**: MountingHole_3.5mm, MountingHole:MountingHole_3.5mm, F.Cu at (91.9, 62.3)
- added REF**: MountingHole_3.5mm, MountingHole:MountingHole_3.5mm, F.Cu at (24.6, 94.0)
Routing:
- net +5V: track 83.1 -> 88.8 mm
- net S3: track 26.8 -> 32.4 mm
- net S4: track 21.0 -> 25.7 mm
- net S1: track 40.4 -> 42.1 mm
- net S2: track 35.9 -> 37.5 mm
- net ADC: track 48.5 -> 49.8 mm
Other:
- board size 76.2 x 53.3 mm -> 76.2 x 55.4 mm
- board text added: "FS-2 Main Telemetry Board Formula Slug V 1.0 Designed By Nathaniel Platt"
