File: Telemetry Board/Telemetry Board.kicad_sch (KiCad schematic)
At the start: 12 parts, among them J1 776180-1, U3 CD74HC4067SM96, U4 ISO1050DUB, U5 NUCLEO-L432KC

Commit message: brakelight ? abd telem board!
Parts:
- added U6: LED Driver, Package_TO_SOT_SMD:SC-74-6_1.55x2.9mm_P0.95mm, symbol FS_3_Global_Symbol_Library:BCR420UE6433HTMA1
Changed lines of the file:
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@@
+	)
+	(symbol
+		(lib_id "FS_3_Global_Symbol_Library:BCR420UE6433HTMA1")
+		(at 224.79 45.72 0)
+		(unit 1)
+		(exclude_from_sim no)
+		(in_bom yes)
+		(on_board yes)
+		(dnp no)
+		(fields_autoplaced yes)
+		(property "Reference" "U6"
+			(at 224.79 35.56 0)
+			(effects
+				(font
+					(size 1.27 1.27)
+				)
+			)
+		)
+		(property "Value" "LED Driver"
+			(at 224.79 38.1 0)
+			(effects
+				(font
+					(size 1.27 1.27)
+				)
+			)
+		)
+		(property "Footprint" "Package_TO_SOT_SMD:SC-74-6_1.55x2.9mm_P0.95mm"
+			(at 225.044 33.274 0)
+			(effects
+				(font
+					(size 1.27 1.27)
+				)
+				(hide yes)
+			)
+		)
+		(property "Datasheet" "https://www.infineon.com/dgdl/Infineon-BCR420U-BCR421U-DataSheet-v02_01-EN.pdf?fileId=5546d4626102d35a01617524f09e061d"
+			(at 224.282 35.306 0)
+			(effects
+				(font
+					(size 1.27 1.27)
+				)
+				(hide yes)
+			)
+		)
+		(property "Description" "LED Driver chip for 10 - 250mA applications. Single driver controlled by Rext"
+			(at 224.028 37.084 0)
+			(effects
+				(font
+					(size 1.27 1.27)
+				)
+				(hide yes)
+			)
+		)
+		(pin "4"
+		)
+		(pin "3"
+		)
+		(pin "1"
+		)
+		(pin "6"
+		)
+		(pin "2"
+		)
+		(pin "5"
+		)
+		(instances
+			(project "Telemetry Board"
+				(path "/dde73ecd-f7ea-407a-a1ab-cf1927044ecb"
+					(reference "U6")
+					(unit 1)
+				)
+			)
+		)
 	)
 	(symbol
